Commit message: Fix mock

File: swervebot_description/urdf/swervebot/swervebot_macro.ros2_control.xacro (robot description, xacro)
@@ -1,5 +1,6 @@
 <?xml version="1.0" encoding="UTF-8"?>
 <robot xmlns:xacro="http://wiki.ros.org/xacro">
-  <xacro:macro name="swervebot_ros2_control" params="
+  <xacro:macro name="swervebot_ros2_control"
+    params="
                name
                prefix
@@ -9,9 +10,10 @@
                sim_gazebo:=false
                simulation_controllers"
-               >
+  >
     <ros2_control name="${name}" type="system">
       <hardware>
         <xacro:if value="${use_mock_hardware}">
           <plugin>mock_components/GenericSystem</plugin>
+          <param name="calculate_dynamics">true</param>
           <param name="mock_sensor_commands">${mock_sensor_commands}</param>
         </xacro:if>
@@ -26,61 +28,44 @@
         </xacro:unless>
       </hardware>
-<!--
       <joint name="${prefix}delta_a">
         <command_interface name="velocity" />
-        <state_interface name="position">
-          <param name="initial_value">0.0</param>
-        </state_interface>
+        <state_interface name="position" />
         <state_interface name="velocity" />
       </joint>
       <joint name="${prefix}delta_b">
-              <command_interface name="velocity" />
-              <state_interface name="position">
-                <param name="initial_value">0.0</param>
-              </state_interface>
-              <state_interface name="velocity" />
+        <command_interface name="velocity" />
+        <state_interface name="position" />
+        <state_interface name="velocity" />
       </joint>
       <joint name="${prefix}delta_c">
-              <command_interface name="velocity" />
-              <state_interface name="position">
-                <param name="initial_value">0.0</param>
-              </state_interface>
-              <state_interface name="velocity" />
+        <command_interface name="velocity" />
+        <state_interface name="position" />
+        <state_interface name="velocity" />
       </joint>
       <joint name="${prefix}delta_d">
-              <command_interface name="velocity" />
-              <state_interface name="position">
-                <param name="initial_value">0.0</param>
-              </state_interface>
-              <state_interface name="velocity" />
+        <command_interface name="velocity" />
+        <state_interface name="position" />
+        <state_interface name="velocity" />
       </joint>
       <joint name="${prefix}gamma_a">
-        <command_interface name="position" />
-        <state_interface name="position">
-          <param name="initial_value">0.0</param>
-        </state_interface>
+        <command_interface name="velocity" />
+        <state_interface name="position" />
         <state_interface name="velocity" />
       </joint>
       <joint name="${prefix}gamma_b">
-              <command_interface name="position" />
-              <state_interface name="position">
-                <param name="initial_value">0.0</param>
-              </state_interface>
-              <state_interface name="velocity" />
+        <command_interface name="velocity" />
+        <state_interface name="position" />
+        <state_interface name="velocity" />
       </joint>
       <joint name="${prefix}gamma_c">
-              <command_interface name="position" />
-              <state_interface name="position">
-                <param name="initial_value">0.0</param>
-              </state_interface>
-              <state_interface name="velocity" />
+        <command_interface name="velocity" />
+        <state_interface name="position" />
+        <state_interface name="velocity" />
       </joint>
       <joint name="${prefix}gamma_d">
-              <command_interface name="position" />
-              <state_interface name="position">
-                <param name="initial_value">0.0</param>
-              </state_interface>
-              <state_interface name="velocity" />
-      </joint> -->
+        <command_interface name="velocity" />
+        <state_interface name="position" />
+        <state_interface name="velocity" />
+      </joint>
     </ros2_control>
     <xacro:if value="$(arg sim_gazebo_classic)">

File: swervebot_description/urdf/swervebot/swervebot_macro.xacro (robot description, xacro)
@@ -4,12 +4,6 @@
   <xacro:include filename="$(find swervebot_description)/urdf/common/materials.xacro" />
   <xacro:macro name="swervebot" params="prefix parent *origin">
-    <link name="${prefix}base_link"></link>
-  <joint name="${parent}_to_${prefix}_base_link" type="fixed">
-    <parent link="${parent}"/>
-    <child link="${prefix}base_link"/>
-    <xacro:insert_block name="origin"/>
-  </joint>
     <joint name="${prefix}base_link_to_base" type="fixed">
-      <parent link="base_link" />
+      <parent link="${prefix}base_link" />
       <child link="chasis" />
       <origin rpy="0.0 0 0" xyz="0 0 0" />
@@ -98,7 +92,7 @@
       <parent link="wheel_anchor" />
       <child link="wheel" />
-      <axis xyz="0 0 1" />
-      <limit effort="1" velocity="20" lower="0" upper="6.283185307179586232" />
-      <joint_properties friction="0.0" />
+       <axis xyz="0 0 1" />
+      <limit effort="1" velocity="20" lower="0" upper="6.283185307179586232" />
+     <joint_properties friction="0.0" />
     </joint>
     <joint name="${prefix}gamma_a" type="revolute">
@@ -331,6 +325,7 @@
       <xacro:insert_block name="origin" />
       <parent link="${parent}" />
-      <child link="base_link" />
-    </joint>
+      <child link="${prefix}base_link" />
+    </joint>
+    <link name="${prefix}base_link"></link>
   </xacro:macro>
 </robot>
